File: pcb/floppa40.kicad_pcb (KiCad board)
At the start: 2 copper layers, 247.5 x 89.2 mm, 46 parts, among them J1 MJ-4PP-9

Commit message: the voices
Parts:
- moved J1 2.29 mm to (128.3, 62.6)
Routing:
- net (no net): track 4307.9 -> 4317.0 mm

Commit message: firm
Routing:
- net (no net): track 4317.0 -> 4311.6 mm

Commit message: real
Parts:
- added G***: LOGO, 42keebs:Powered_by_QMK-25mm-SilkS, F.Cu at (215.9, 74.4)
- added G***: LOGO, 42keebs:osh-logo, F.Cu at (215.1, 68.3)

Commit message: :|
Parts:
- added REF**: MountingHole_3.2mm_M3, MountingHole:MountingHole_3.2mm_M3, F.Cu at (181.6, 70.4)
- added REF**: MountingHole_3.2mm_M3, MountingHole:MountingHole_3.2mm_M3, F.Cu at (202.2, 144.8)
- added REF**: MountingHole_3.2mm_M3, MountingHole:MountingHole_3.2mm_M3, F.Cu at (238.8, 144.5)
- added REF**: MountingHole_3.2mm_M3, MountingHole:MountingHole_3.2mm_M3, F.Cu at (26.9, 123.4)
- added REF**: MountingHole_3.2mm_M3, MountingHole:MountingHole_3.2mm_M3, F.Cu at (120.9, 63.8)
- added REF**: MountingHole_3.2mm_M3, MountingHole:MountingHole_3.2mm_M3, F.Cu at (30.2, 69.8)
- added farted: Choc, 42keebs:Kailh_socket_PG1350_2u_Stabilizer, F.Cu at (252.0, 107.1)
- added farted: Choc, 42keebs:Kailh_socket_PG1350_2u_Stabilizer, F.Cu at (177.8, 141.1)
- added farted: Choc, 42keebs:Kailh_socket_PG1350_2u_Stabilizer, F.Cu at (110.2, 141.1)
Routing:
- net (no net): track 4311.6 -> 4326.4 mm

Commit message: real
Parts:
- removed the G*** at (215.1, 68.3)
- added REF**: OSHW-Symbol_6.7x6mm_SilkScreen, Symbol:OSHW-Symbol_6.7x6mm_SilkScreen, F.Cu at (209.0, 69.6)
- moved G*** 0.80 mm to (215.6, 75.2)

Commit message: centered i think
Parts:
- moved REF** 1.92 mm to (208.6, 67.7)
- moved G*** 1.92 mm to (215.2, 73.3)

Commit message: based keyboard man thank
Routing:
- net (no net): track 4326.4 -> 4325.5 mm
Other:
- rule pad_to_mask_clearance: 0 -> 0.05
